File: board/board.kicad_pcb (KiCad board)
At the start: 2 copper layers, 37.1 x 49.8 mm, 13 parts, among them J1 Conn_01x19, J2 Conn_01x19, J3 3.3-26V, U1 ESP32-WROVER-E, U2 AOZ1280CI

Commit message: dev
Parts:
- added J4: Conn_01x19, Connector_PinHeader_1.27mm:PinHeader_1x19_P1.27mm_Vertical, F.Cu at (144.9, 54.6)
- added J5: Conn_01x19, Connector_PinHeader_1.27mm:PinHeader_1x19_P1.27mm_Vertical, F.Cu at (162.4, 54.6)

Commit message: dev
Parts:
- C1: renamed from C2; footprint Capacitor_SMD:C_1206_3216Metric -> Capacitor_Tantalum_SMD:CP_EIA-7343-31_Kemet-D_Pad2.25x2.55mm_HandSolder
- J1: renamed from J3; value 3.3-26V -> 5-26V
- L1: footprint Inductor_SMD:L_1206_3216Metric -> Custom_Inductor:Shielded_3.0_3.0
- R1: renamed from R3; value R_Small -> 100k - 600k
- moved C1 3.60 mm to (154.8, 97.8), turned to -90 degrees
- moved R2 2.24 mm to (145.9, 90.6)
- moved C3 2.04 mm to (145.9, 87.2)
- moved R3 1.75 mm to (150.0, 92.5), turned to -90 degrees
- moved L1 1.50 mm to (145.9, 83.4)
- renumbered C3 to C2, C4 to C3, J1 to J2, J4 to J3, J5 to J4, J2 to J5, R1 to R2, R2 to R3, U2 to U1, U1 to U2
Routing:
- net 3.3: track 37.9 -> 39.3 mm, vias 0 -> 6
- net GND: vias 46 -> 96
- net /VOUT: vias 0 -> 10
- net /VIN: vias 14 -> 22
- added copper zone on B.Cu, net /VOUT
- added copper zone on B.Cu, net 3.3
